Commit message: Added updated package odom exists

File: amr/urdf/amr_st.urdf (robot description, URDF)
Before this commit: robot mogi_bot, 7 links, 6 joints
Links:
- removed link imu_link
- link base_link: mass 24.18896015187 -> 24.189; geometry collision mesh filename=package://amr/meshes/backup_files/base_link.STL; visual mesh filename=package://amr/meshes/backup_files/base_link.STL
- link bl_link: mass None -> 2.1167; geometry collision mesh filename=package://amr/meshes/backup_files/bl_link.STL; visual mesh filename=package://amr/meshes/backup_files/bl_link.STL
- link br_link: mass None -> 2.11669573162388; geometry collision mesh filename=package://amr/meshes/backup_files/br_link.STL; visual mesh filename=package://amr/meshes/backup_files/br_link.STL
- link cam_link: mass 0.2379 -> 0.23789184766465; geometry collision mesh filename=package://amr/meshes/backup_files/cam_link.STL; visual mesh filename=package://amr/meshes/backup_files/cam_link.STL
- link scan_link: geometry collision mesh filename=package://amr/meshes/backup_files/scan_link.STL; visual mesh filename=package://amr/meshes/backup_files/scan_link.STL
Joints:
- removed joint imu_joint
- joint cam_joint: axis (none) -> 0 0 0; limit (none) -> effort=100 velocity=10; origin xyz=0.45 -0.0034 0.0296 rpy=0 0 0 -> xyz=0.45 -0.0033621 0.029649 rpy=0 0 0
- joint left_wheel_joint: axis 0 1 0 -> 0 -1 0; origin xyz=-0.2 0.325 0.03 rpy=0 0 0 -> xyz=-0.2 0.325 0.03 rpy=0 0 3.14159265358979
- joint scan_joint: origin xyz=0.2624 0 0.1025 rpy=0 0 0 -> xyz=0.26245 0 0.1025 rpy=0 0 0; type continuous -> fixed

Commit message: added

File: amr/urdf/amr_st.urdf (robot description, URDF)
Before this commit: robot amr, 6 links, 5 joints
Links:
- removed link bl_link
- removed link br_link
- removed link cam_link
- added link camera_link, mass 0; collision mesh filename=package://amr/meshes/camera_link.STL; visual mesh filename=package://amr/meshes/camera_link.STL
- added link camera_link_optical
- added link imu_link
- added link left_wheel, mass 1.5707963267949; collision mesh filename=package://amr/meshes/left_wheel.STL; visual mesh filename=package://amr/meshes/left_wheel.STL
- added link right_wheel, mass 1.5707963267949; collision mesh filename=package://amr/meshes/right_wheel.STL; visual mesh filename=package://amr/meshes/right_wheel.STL
- link base_link: mass 24.189 -> 7.5204; geometry collision mesh filename=package://amr/meshes/base_link.STL; visual mesh filename=package://amr/meshes/base_link.STL
- link scan_link: mass 1.1486 -> 0.392699081698724; geometry collision mesh filename=package://amr/meshes/scan_link.STL; visual mesh filename=package://amr/meshes/scan_link.STL
Joints:
- removed joint cam_joint
- added joint camera_joint: type fixed, parent base_link, child camera_link, origin xyz=-0.00250000000000108 -0.175 -0.0375000000000026 rpy=0 0 0, axis 0 0 0
- added joint camera_optical_joint: type fixed, parent camera_link, child camera_link_optical, origin xyz=0 0 0 rpy=-1.5707 0 -1.5707
- added joint imu_joint: type fixed, parent base_link, child imu_link, origin xyz=0 0 0 rpy=0 0 0
- joint left_wheel_joint: axis 0 -1 0 -> 1 0 0; child bl_link -> left_wheel; limit effort=100 velocity=10 -> (none); origin xyz=-0.2 0.325 0.03 rpy=0 0 3.14159265358979 -> xyz=0.13 0 -0.075 rpy=0 0 0
- joint right_wheel_joint: axis 0 1 0 -> 1 0 0; child br_link -> right_wheel; limit effort=100 velocity=10 -> (none); origin xyz=-0.2 -0.325 0.03 rpy=0 0 0 -> xyz=-0.13 0 -0.075 rpy=0 0 0
- joint scan_joint: origin xyz=0.26245 0 0.1025 rpy=0 0 0 -> xyz=-0.00055325 -0.075003 0.025 rpy=0 0 0; type fixed -> continuous
